File: main.kicad_pcb (KiCad board)
At the start: 2 copper layers, 24 parts, among them SW1 SW_Push, U1 ATmega32U4-A, Y1 16MHz

Commit message: some bad routing
Parts:
- moved C1 0.95 mm to (140.1, 83.0)
- moved R3 0.18 mm to (124.0, 72.9), turned to -90 degrees
Connections:
- C6 pad 2: Net-(U1-XTAL2) -> Net-(U1-XTAL1)
- C7 pad 2: Net-(U1-AREF) -> Net-(U1-XTAL2)
- U1 pad 17: unconnected-(U1-XTAL1-Pad17) -> Net-(U1-XTAL1)
- U1 pad 42: Net-(U1-AREF) -> unconnected-(U1-AREF-Pad42)
- Y1 pad 1: Net-(U1-XTAL2) -> Net-(U1-XTAL1)
- Y1 pad 3: Net-(U1-AREF) -> Net-(U1-XTAL2)
Routing:
- net GND: track 0.00 -> 130.5 mm
- net +5V: track 0.00 -> 87.7 mm
- net Net-(U1-~{RESET}): track 0.00 -> 54.2 mm
- net Net-(U1-D-): track 0.00 -> 25.7 mm
- net Net-(U1-D+): track 0.00 -> 21.6 mm
- net ROW0: track 0.00 -> 19.2 mm
- net ROW1: track 0.00 -> 19.2 mm
- net VCC: track 0.00 -> 12.3 mm
- net Net-(U1-XTAL2): track 0.00 -> 11.0 mm
- net Net-(U1-XTAL1): track 0.00 -> 8.98 mm
- net Net-(D4-A): track 0.00 -> 7.02 mm
- net Net-(D3-A): track 0.00 -> 7.02 mm
- net Net-(D1-A): track 0.00 -> 7.02 mm
- net Net-(D2-A): track 0.00 -> 7.02 mm
- net D+: track 0.00 -> 5.61 mm
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