File: main.kicad_sch (KiCad schematic)
At the start: 14 parts, among them SW1 SW_Push, U1 ATmega32U4-A, Y1 16MHz

Commit message: beginning board design
Parts:
- added D1, D2, D3, D4: D_Small, Diode_SMD:D_SOD-123, symbol Device:D_Small
- added F1: 500mA, Fuse:Fuse_1206_3216Metric, symbol Device:Polyfuse_Small
- added MX1, MX2, MX3, MX4: MX-NoLED, MX_Alps_Hybrid:MX-1U-NoLED, symbol MX_Alps_Hybrid:MX-NoLED
- added USB1: Molex-0548190589, random-keyboard-parts:Molex-0548190589, symbol random-keyboard-parts:Molex-0548190589
- C1, C2, C3, C4, C5, C6, C7: footprint (none) -> Capacitor_SMD:C_0805_2012Metric
- R1, R2, R3, R4: footprint (none) -> Resistor_SMD:R_0805_2012Metric
- SW1: footprint (none) -> random-keyboard-parts:SKQG-1155865
- Y1: footprint (none) -> Crystal:Crystal_SMD_3225-4Pin_3.2x2.5mm
Connections:
- net +5V: now also F1.2
- net D+: now also USB1.3 (D+)
- net D-: now also USB1.4 (D-)
- net GND: now also USB1.1 (GND)
- net at C6.2, U1.16 (XTAL2): now also Y1.1; no longer Y1.3
- net at C7.2, U1.42 (AREF): now also Y1.3; no longer Y1.1
- new net: D4.2 (A), MX4.2 (ROW)
- new net: D1.2 (A), MX1.2 (ROW)
- new net: D3.2 (A), MX3.2 (ROW)
- new net: D2.2 (A), MX2.2 (ROW)
- new net COL0: MX1.1 (COL), MX3.1 (COL)
- new net COL1: MX2.1 (COL), MX4.1 (COL)
- new net ROW0: D1.1 (K), D2.1 (K)
- new net ROW1: D3.1 (K), D4.1 (K)
- new net VCC: F1.1, USB1.5 (VBUS)
Other:
- moved on the sheet: Y1

Commit message: some bad routing
Connections:
- net at C6.2, Y1.1: now also U1.17 (XTAL1); no longer U1.16 (XTAL2)
- net at C7.2, Y1.3: now also U1.16 (XTAL2); no longer U1.42 (AREF)
Changed lines of the file:
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@@
 	(paper "A4")
 	(junction
+		(at 107.95 72.39)
+		(diameter 0)
+		(color 0 0 0 0)
+	)
+	(junction
 		(at 57.15 154.94)
 		(diameter 0)
@@
 	)
 	(junction
-		(at 107.95 72.39)
+		(at 107.95 77.47)
 		(diameter 0)
 		(color 0 0 0 0)
@@
 	)
 	(junction
-		(at 107.95 77.47)
-		(diameter 0)
-		(color 0 0 0 0)
-	)
-	(junction
 		(at 104.14 124.46)
 		(diameter 0)
@@
 	(wire
 		(pts
-			(xy 107.95 77.47) (xy 135.89 77.47)
+			(xy 115.57 73.66) (xy 135.89 73.66)
 		)
 		(stroke
@@
 	(wire
 		(pts
+			(xy 115.57 77.47) (xy 115.57 73.66)
+		)
+		(stroke
+			(width 0)
+			(type default)
+		)
+	)
+	(wire
+		(pts
 			(xy 93.98 124.46) (xy 99.06 124.46)
 		)
@@
 	(wire
 		(pts
+			(xy 107.95 77.47) (xy 115.57 77.47)
+		)
+		(stroke
+			(width 0)
+			(type default)
+		)
+	)
+	(wire
+		(pts
 			(xy 110.49 74.93) (xy 110.49 81.28)
 		)
@@
 	(wire
 		(pts
+			(xy 102.87 72.39) (xy 107.95 72.39)
+		)
+		(stroke
+			(width 0)
+			(type default)
+		)
+	)
+	(wire
+		(pts
 			(xy 107.95 90.17) (xy 135.89 90.17)
 		)
@@
 	(wire
 		(pts
+			(xy 135.89 73.66) (xy 135.89 72.39)
+		)
+		(stroke
+			(width 0)
+			(type default)
+		)
+	)
+	(wire
+		(pts
 			(xy 34.29 165.1) (xy 46.99 165.1)
 		)
@@
 	(wire
 		(pts
-			(xy 102.87 72.39) (xy 107.95 72.39)
+			(xy 125.73 67.31) (xy 135.89 67.31)
 		)
 		(stroke
@@
 	(wire
 		(pts
-			(xy 107.95 72.39) (xy 135.89 72.39)
+			(xy 107.95 72.39) (xy 125.73 72.39)
 		)
 		(stroke
@@
 		)
 		(stroke
+			(width 0)
+			(type default)
+		)
+	)
+	(wire
+		(pts
+			(xy 125.73 72.39) (xy 125.73 67.31)
+		)
+		(stroke
